Commit message: feat: added cool race car model

File: simulation/models/robot/robot.urdf (robot description, URDF)
Before this commit: robot race_robot, 6 links, 5 joints
Links:
- link base_link: geometry collision box size=0.22 0.18 0.06; visual box size=0.004 0.035 0.012
- link left_wheel_link: geometry collision cylinder length=0.025 radius=0.035; visual box size=0.012 0.028 0.008
- link right_wheel_link: geometry collision cylinder length=0.025 radius=0.035; visual box size=0.012 0.028 0.008
